File: ESP32Breakout/ESP32Breakout/ESP32Breakout.kicad_pcb (KiCad board)
At the start: 2 copper layers, 100 x 60 mm, 45 parts, among them J1 Conn_01x15_Socket, J10 RESET, J11 START, J12 PAUSE, J13 TIME SEL, J14 LED0, J15 LED1, J16 LED2, J17 LED3, J18 Conn_01x09_Pin, J19 Conn_01x07_Pin, J2 Conn_01x15_Socket, J3 5V INPUT, J4 Bell Power, J5 Screw_Terminal_01x03, J6 Screw_Terminal_01x03, J7 Bell Power, J8 Screw_Terminal_01x03, J9 Screw_Terminal_01x03, K1 G5V-2_Split, K2 G5V-2_Split, Q1 BSS214NW, Q2 BSS214NW, SW1 RESET, SW2 START, SW3 PAUSE, SW4 SW_SPDT

Commit message: update production files for both boards
Parts:
- removed the ? at (149.3, 90.0)
- removed the ? at (149.3, 38.0)
- removed the ? at (57.3, 90.0)
- added ?: , , F.Cu at (57.3, 90.0)
- added ?: , , F.Cu at (149.2, 38.0)
- added REF**: MountingHole_3.2mm_M3, MountingHole:MountingHole_3.2mm_M3, F.Cu at (149.3, 90.0)
Connections:
- net nPAUSE renamed nBTN3
- net nRESET renamed nBTN1
- net nSTART renamed nBTN2
Other:
- board text added: "SEMO Combat Robtics 2024 Vinnie Marco Mitch Cerroni"
- board text removed: "Vinnie Marco Mitch Cerroni SEMO Combat Robtics 2024"
