File: ArenaTimer/ArenaTimer.kicad_pcb (KiCad board)
At the start: 2 copper layers, 262.3 x 230 mm, 179 parts, among them J1 POWER IN, J2 Conn_01x02_Pin, J3 Conn_01x02_Pin, J4 GND, J5 5V, J6 GND, J7 5V

Commit message: update board outline, generate production files
Parts:
- added ?: , , F.Cu at (55.8, 225.4)
- added ?: , , F.Cu at (55.8, 55.4)
- added ?: , , F.Cu at (161.9, 55.4)
- added ?: , , F.Cu at (55.8, 140.4)
- added ?: , , F.Cu at (161.9, 225.4)
- added ?: , , F.Cu at (158.1, 140.4)
- added REF**: MountingHole_3.2mm_M3_DIN965, MountingHole:MountingHole_3.2mm_M3_DIN965, F.Cu at (268.1, 55.4)
- added REF**: MountingHole_3.2mm_M3_DIN965, MountingHole:MountingHole_3.2mm_M3_DIN965, F.Cu at (268.1, 140.4)
- added REF**: MountingHole_3.2mm_M3_DIN965, MountingHole:MountingHole_3.2mm_M3_DIN965, F.Cu at (268.1, 225.4)
- moved J4 15.1 mm to (268.4, 40.7)
- moved J6 15.0 mm to (268.4, 232.3)
- moved J7 6.46 mm to (268.4, 62.5)
- moved J5 6.36 mm to (268.4, 210.5)
- moved JP1 6.16 mm to (282.9, 88.3)
- moved J2 5.49 mm to (268.4, 78.8)
- moved J3 5.39 mm to (268.4, 201.8)
- moved J1 0.52 mm to (266.7, 151.8)
Routing:
- net /TimerBorder/DIN: track 62.5 -> 71.6 mm
- net /TimerDigit6/DIN: track 212.6 -> 206.0 mm
- net /TimerColon/DOUT: track 155.3 -> 149.2 mm
- net /TimerBorder/DOUT: track 48.3 -> 53.9 mm
- net /TimerDigit/DIN: track 117.2 -> 119.2 mm
Other:
- board size 262.3 x 230 mm -> 262.2 x 230 mm
- board text added: "BIN"
- board text added: "BOUT"
- board text added: "DIN"
- board text added: "DOUT"
- board text removed: "BDR IN"
- board text removed: "BORDER OUT"
- board text removed: "DIGIT IN"
- board text removed: "DIGIT OUT"

Commit message: update production files for both boards
Other:
- board text added: "SEMO Combat Robotics 2024 Vinnie Marco Mitch Cerroni"
Changed lines of the file:
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@@
 		(tags "solder jumper open")
 		(property "Reference" "JP1"
-			(at -2.9464 0.0508 360)
+			(at -2.9464 0.0508 0)
 			(layer "F.SilkS")
 			(effects
@@
 		)
 		(property "Value" "Jumper_2_Open"
-			(at 0 1.9 360)
+			(at 0 1.9 0)
 			(layer "F.Fab")
 			(effects
@@
 		(tags "Through hole pin header THT 1x02 2.54mm single row")
 		(property "Reference" "J3"
-			(at -2.54 0.0304 360)
+			(at -2.54 0.0304 0)
 			(layer "F.SilkS")
 			(hide yes)
@@
 		)
 		(property "Value" "Conn_01x02_Pin"
-			(at 0 4.87 360)
+			(at 0 4.87 0)
 			(layer "F.Fab")
 			(effects
@@
 		(tags "Through hole pin header THT 1x04 2.54mm single row")
 		(property "Reference" "J6"
-			(at 0 -2.33 360)
+			(at 0 -2.33 0)
 			(layer "F.SilkS")
 			(hide yes)
@@
 		)
 		(property "Value" "GND"
-			(at 0 9.95 360)
+			(at 0 9.95 0)
 			(layer "F.Fab")
 			(effects
@@
 		(tags "Through hole pin header THT 1x04 2.54mm single row")
 		(property "Reference" "J5"
-			(at 0 -2.33 360)
+			(at 0 -2.33 0)
 			(layer "F.SilkS")
 			(hide yes)
@@
 		)
 		(property "Value" "5V"
-			(at 0 9.95 360)
+			(at 0 9.95 0)
 			(layer "F.Fab")
 			(effects
@@
 		(layer "Edge.Cuts")
 	)
+	(gr_text "SEMO Combat Robotics 2024\nVinnie Marco\nMitch Cerroni"
+		(at 262.9154 52.1208 0)
+		(layer "B.SilkS")
+		(effects
+			(font
+				(size 5 5)
+				(thickness 1.25)
+				(bold yes)
+			)
+			(justify left bottom mirror)
+		)
+	)
 	(gr_text "Short JP1 to put border \nin serial with digits"

Commit message: add 3d models
Parts:
- removed ? (x6): , 
- removed REF** (x3): MountingHole_3.2mm_M3_DIN965, MountingHole:MountingHole_3.2mm_M3_DIN965
- added D40: 1N1007, SMA, Diode_SMD:D_SMA, F.Cu at (58.9, 83.0)
- added H1: MountingHole, MountingHole:MountingHole_3.2mm_M3, F.Cu at (55.8, 55.4)
- added H2: MountingHole, MountingHole:MountingHole_3.2mm_M3, F.Cu at (55.8, 140.4)
- added H3: MountingHole, MountingHole:MountingHole_3.2mm_M3, F.Cu at (55.8, 225.4)
- added H4: MountingHole, MountingHole:MountingHole_3.2mm_M3, F.Cu at (161.9, 55.4)
- added H5: MountingHole, MountingHole:MountingHole_3.2mm_M3, F.Cu at (158.0, 140.4)
- added H6: MountingHole, MountingHole:MountingHole_3.2mm_M3, F.Cu at (161.9, 225.4)
- added H7: MountingHole, MountingHole:MountingHole_3.2mm_M3, F.Cu at (268.0, 55.4)
- added H8: MountingHole, MountingHole:MountingHole_3.2mm_M3, F.Cu at (268.0, 140.4)
- added H9: MountingHole, MountingHole:MountingHole_3.2mm_M3, F.Cu at (268.0, 225.4)
- added J10: Red ready-up, Connector_JST:JST_EH_S2B-EH_1x02_P2.50mm_Horizontal, B.Cu at (239.4, 248.6)
- added J11: Bell Power, TerminalBlock:TerminalBlock_bornier-2_P5.08mm, B.Cu at (40.4, 29.2)
- added J12: Screw_Terminal_01x03, TerminalBlock:TerminalBlock_bornier-3_P5.08mm, B.Cu at (74.6, 29.2)
- added J13: Screw_Terminal_01x03, TerminalBlock:TerminalBlock_bornier-3_P5.08mm, B.Cu at (55.1, 29.2)
- added J15: Conn_01x15_Socket, Connector_PinSocket_2.54mm:PinSocket_1x15_P2.54mm_Vertical, B.Cu at (122.8, 164.8)
- added J16: Conn_01x15_Socket, Connector_PinSocket_2.54mm:PinSocket_1x15_P2.54mm_Vertical, B.Cu at (122.8, 190.2)
- added J8: Barrel_Jack, Connector_BarrelJack:BarrelJack_Horizontal, B.Cu at (63.0, 243.6)
- added J9: Conn_01x06_Pin, Connector_JST:JST_EH_S6B-EH_1x06_P2.50mm_Horizontal, B.Cu at (256.9, 248.6)
- added K1: G5V-2_Split, Relay_THT:Relay_DPDT_Omron_G5V-2, F.Cu at (62.8, 79.2)
- added Q1: BSS214NW, Package_TO_SOT_SMD:SOT-323_SC-70, F.Cu at (56.7, 86.5)
- added R2: 100K, Resistor_SMD:R_0402_1005Metric, F.Cu at (56.6, 88.8)
- J1: value POWER IN -> Blue ready-up; footprint TerminalBlock:TerminalBlock_Altech_AK300-2_P5.00mm -> Connector_JST:JST_EH_S2B-EH_1x02_P2.50mm_Horizontal; moved to B.Cu
- J2: value Conn_01x02_Pin -> Conn_01x02_Socket; footprint Connector_PinHeader_2.54mm:PinHeader_1x02_P2.54mm_Vertical -> Connector_PinSocket_2.54mm:PinSocket_1x02_P2.54mm_Horizontal; moved to B.Cu
- J3: footprint Connector_PinHeader_2.54mm:PinHeader_1x02_P2.54mm_Vertical -> Connector_PinHeader_2.54mm:PinHeader_1x02_P2.54mm_Horizontal; moved to B.Cu
- J4, J5: footprint Connector_PinHeader_2.54mm:PinHeader_1x04_P2.54mm_Vertical -> Connector_PinHeader_2.54mm:PinHeader_1x04_P2.54mm_Horizontal; moved to B.Cu
- J6, J7: footprint Connector_PinHeader_2.54mm:PinHeader_1x04_P2.54mm_Vertical -> Connector_PinSocket_2.54mm:PinSocket_1x04_P2.54mm_Horizontal; moved to B.Cu
- JP1: moved to B.Cu
- moved JP1 248.3 mm to (39.7, 38.4), turned to 180 degrees
- moved J1 106.9 mm to (221.2, 248.6), turned to 0 degrees
- moved J5 8.11 mm to (265.9, 218.3)
- moved J4 8.00 mm to (265.9, 48.3)
- moved J3 3.59 mm to (266.0, 204.5)
- moved J2 3.54 mm to (265.9, 76.3)
- moved J7 2.44 mm to (265.9, 62.5), turned to 180 degrees
- moved J6 2.39 mm to (266.0, 232.4), turned to 180 degrees
Connections:
- D252 pad 4: /TimerBorder/DIN -> BORDER_LEDS
- D329 pad 4: /TimerDigit6/DIN -> DIGIT_LEDS
- J1 pad 1: GND -> nBLUE_RDY_BTN
- J1 pad 2: +5V -> GND
- J2 pad 1: /TimerDigit6/DIN -> BORDER_LEDS
- J2 pad 2: /TimerBorder/DIN -> DIGIT_LEDS
- JP1 pad 1: /TimerBorder/DIN -> Net-(J11-Pin_1)
- JP1 pad 2: /TimerColon/DOUT -> +5V
Routing:
- net BORDER_LEDS: track 0.00 -> 358.3 mm, vias 0 -> 3
- net DIGIT_LEDS: track 0.00 -> 331.3 mm, vias 0 -> 2
- net nTIME_SEL: track 0.00 -> 248.6 mm, vias 0 -> 2
- net nRESET_BTN: track 0.00 -> 246.0 mm, vias 0 -> 2
- net nPAUSE_BTN: track 0.00 -> 241.2 mm, vias 0 -> 2
- net nSTART_BTN: track 0.00 -> 237.5 mm, vias 0 -> 2
- net nBUZZER_BTN: track 0.00 -> 224.9 mm, vias 0 -> 2
- net /TimerDigit6/DIN: track 206.0 -> 0.00 mm, vias 15 -> 0
- net RELAY_EN: track 0.00 -> 129.2 mm, vias 0 -> 1
- net /TimerBorder/DIN: track 71.6 -> 0.00 mm
- net Net-(J11-Pin_1): track 0.00 -> 59.7 mm
- net Net-(J12-Pin_1): track 0.00 -> 44.2 mm
- net Net-(J13-Pin_1): track 0.00 -> 40.9 mm
- net Net-(J12-Pin_2): track 0.00 -> 40.6 mm
- net Net-(J13-Pin_2): track 0.00 -> 34.3 mm
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Other:
- board text added: "+5V Input Only!"
- board text added: "BUZZER"
- board text added: "Blue Rdy"
- board text added: "Do not populate J2 on host side"
- board text added: "ESP32 Module"
- board text added: "ESP32, Power Jack, Relay, and screw terminals only need to be popluated one one board per timer!"
- board text added: "NC"
- board text added: "NO"
- board text added: "PAUSE"
- board text added: "RESET"
- board text added: "Red Rdy"
- board text added: "SEMO Combat Robotics 2025 Vinnie Marco Mitch Cerroni"
- board text added: "START"
- board text added: "Short JP1 for 5V buzzer power"
- board text added: "TIME SEL"
- board text added: "V+"
- board text removed: "SEMO Combat Robotics 2024 Vinnie Marco Mitch Cerroni"
- board text removed: "Short JP1 to put border in serial with digits"
