File: ArenaTimer/TimerBorder.kicad_sch (KiCad schematic)
At the start: 72 parts

Commit message: added digits
Parts:
- renumbered C181 to C1, C190 to C100, C191 to C101, C192 to C102, C193 to C103, C194 to C104, C209 to C105, C195 to C106, C196 to C107, C210 to C108, C197 to C109, C198 to C110, C211 to C111, C199 to C112, C200 to C113, C212 to C114, C201 to C115, C202 to C116, C213 to C117, C203 to C118, C204 to C119, C214 to C120, C205 to C121, C206 to C122, C215 to C123, C207 to C124, C208 to C125, C216 to C126, C182 to C92, C183 to C93, C184 to C94, C185 to C95, C186 to C96, C187 to C97, C188 to C98, C189 to C99, D181 to D1, D190 to D100, D191 to D101, D192 to D102, D193 to D103, D194 to D104, D209 to D105, D195 to D106, D196 to D107, D210 to D108, D197 to D109, D198 to D110, D211 to D111, D199 to D112, D200 to D113, D212 to D114, D201 to D115, D202 to D116, D213 to D117, D203 to D118, D204 to D119, D214 to D120, D205 to D121, D206 to D122, D215 to D123, D207 to D124, D208 to D125, D216 to D126, D182 to D92, D183 to D93, D184 to D94, D185 to D95, D186 to D96, D187 to D97, D188 to D98, D189 to D99

Commit message: finish up routing
Parts:
- removed C1, C100, C101, C102, C103, C104, C105, C106, C107, C108, C109, C110, C111, C112, C113, C114, C115, C116, C117, C118, C119, C120, C121, C122, C123, C124, C125, C126, C92, C93, C94, C95, C96, C97, C98, C99: 100nF, symbol Device:C
- removed D1, D100, D101, D102, D103, D104, D105, D106, D107, D108, D109, D110, D111, D112, D113, D114, D115, D116, D117, D118, D119, D120, D121, D122, D123, D124, D125, D126, D92, D93, D94, D95, D96, D97, D98, D99: WS2812B, LED_SMD:LED_WS2812B_PLCC4_5.0x5.0mm_P3.2mm, symbol LED:WS2812B
Other:
- added sheet TimerQuadrant (timerquadrant.kicad_sch)
- added sheet TimerQuadrant1 (timerquadrant.kicad_sch)
- note added: "Front Side"
- note removed: "36 LEDs, can make more hierarchical to increase LED count"
