File: ArenaTimer/TimerColon.kicad_sch (KiCad schematic)
At the start: 12 parts

Commit message: finish up routing
Parts:
- removed C30, C31, C32, C33, C34, C35: 100nF, symbol Device:C
- removed D33, D34, D35: WS2812B, LED_SMD:LED_WS2812B_PLCC4_5.0x5.0mm_P3.2mm, symbol LED:WS2812B
- renumbered D30 to D1, D31 to D2, D32 to D3
Connections:
- net DOUT: now also D3.2 (DOUT)
Other:
- note added: "Colon"
- note removed: "Bottom Dot"
- note removed: "Top Dot"
- moved on the sheet: D1, D2, D3
